Commit message: spiderx_description: add sim_backend switch, lidar_link and Fortress extensions
- sim_backend xacro arg (classic|fortress|none). The default, classic,
  expands to the same URDF as before apart from the new lidar link, so
  the legacy Gazebo Classic path and display.launch.py are unaffected.
  Invalid values fail with xacro.fatal.
- lidar_link + fixed lidar_joint on base_link, placed on the measured
  top-plate centre/top surface. Mass/inertia are labelled
  SIMULATION_ESTIMATE.
- spiderx_fortress.gazebo.xacro: gpu_lidar (360 x 1 deg, 0.15-12 m,
  10 Hz, ignition_frame_id=lidar_link), the JointStatePublisher system,
  and the same contact parameters as the legacy spiderx.gazebo.
- The 8 placeholder horn inertias are labelled; no CAD value changed.

Co-Authored-By: Claude Opus 5.5 <noreply@anthropic.com>
Claude-Session: https://claude.ai/code/session_01QzFL2kguRig19KtzFfqEm3

File: src/spiderx_description/urdf/spiderx.urdf.xacro (robot description, xacro)
@@ -1,7 +1,24 @@
 <?xml version="1.0" ?>
 <robot name="spiderx" xmlns:xacro="http://www.ros.org/wiki/xacro">
+<!-- sim_backend selects which simulator-specific extensions are merged into this
+     description. Geometry, inertia and kinematics are identical for every value.
+       classic  : legacy Gazebo Classic tags (spiderx.trans + spiderx.gazebo).
+                  Default, so existing Classic/RViz users get the previous output.
+       fortress : Gazebo Fortress (Ignition Gazebo 6) sensor/systems only
+                  (spiderx_fortress.gazebo.xacro). No Gazebo Classic plugins.
+       none     : no simulator tags (RViz, hardware bring-up). -->
+<xacro:arg name="sim_backend" default="classic" />
+<xacro:property name="sim_backend" value="$(arg sim_backend)" />
+<xacro:unless value="${sim_backend in ['classic', 'fortress', 'none']}">
+  ${xacro.fatal("sim_backend must be 'classic', 'fortress' or 'none', got '" + sim_backend + "'")}
+</xacro:unless>
 <xacro:include filename="$(find spiderx_description)/urdf/materials.xacro" />
-<xacro:include filename="$(find spiderx_description)/urdf/spiderx.trans" />
-<xacro:include filename="$(find spiderx_description)/urdf/spiderx.gazebo" />
+<xacro:if value="${sim_backend == 'classic'}">
+  <xacro:include filename="$(find spiderx_description)/urdf/spiderx.trans" />
+  <xacro:include filename="$(find spiderx_description)/urdf/spiderx.gazebo" />
+</xacro:if>
+<xacro:if value="${sim_backend == 'fortress'}">
+  <xacro:include filename="$(find spiderx_description)/urdf/spiderx_fortress.gazebo.xacro" />
+</xacro:if>
 <link name="dummy_link">
 </link>
@@ -114,4 +131,6 @@
     <origin xyz="1.9542700790964318e-13 0.0002969285186710108 -9.71445146547012e-17" rpy="0 0 0"/>
     <mass value="0.004911019644749942"/>
+    <!-- PLACEHOLDER inertia, not CAD-exact (CAD ~1.2e-7..2.3e-7 was rounded to 0 by the
+         exporter). Physically valid; kept unchanged. See docs/URDF_INERTIA_AUDIT.md -->
     <inertia ixx="1e-6" iyy="1e-6" izz="1e-6" ixy="-0.0" iyz="-0.0" ixz="0.0"/>
   </inertial>
@@ -134,4 +153,6 @@
     <origin xyz="1.9533680228889239e-13 0.00029692851867103853 -1.249000902703301e-16" rpy="0 0 0"/>
     <mass value="0.004911019644749942"/>
+    <!-- PLACEHOLDER inertia, not CAD-exact (CAD ~1.2e-7..2.3e-7 was rounded to 0 by the
+         exporter). Physically valid; kept unchanged. See docs/URDF_INERTIA_AUDIT.md -->
     <inertia ixx="1e-6" iyy="1e-6" izz="1e-6" ixy="-0.0" iyz="-0.0" ixz="0.0"/>
   </inertial>
@@ -154,4 +175,6 @@
     <origin xyz="1.9531598560718066e-13 -0.000296928518671042 -1.1102230246251565e-16" rpy="0 0 0"/>
     <mass value="0.004911019644749942"/>
+    <!-- PLACEHOLDER inertia, not CAD-exact (CAD ~1.2e-7..2.3e-7 was rounded to 0 by the
+         exporter). Physically valid; kept unchanged. See docs/URDF_INERTIA_AUDIT.md -->
     <inertia ixx="1e-6" iyy="1e-6" izz="1e-6" ixy="0.0" iyz="0.0" ixz="0.0"/>
   </inertial>
@@ -174,4 +197,6 @@
     <origin xyz="1.9534547590627227e-13 -0.00029692851867095527 -9.71445146547012e-17" rpy="0 0 0"/>
     <mass value="0.004911019644749942"/>
+    <!-- PLACEHOLDER inertia, not CAD-exact (CAD ~1.2e-7..2.3e-7 was rounded to 0 by the
+         exporter). Physically valid; kept unchanged. See docs/URDF_INERTIA_AUDIT.md -->
     <inertia ixx="1e-6" iyy="1e-6" izz="1e-6" ixy="0.0" iyz="0.0" ixz="0.0"/>
   </inertial>
@@ -354,4 +379,6 @@
     <origin xyz="-0.0002969285186709414 1.3877787807814457e-16 -1.9548251906087444e-13" rpy="0 0 0"/>
     <mass value="0.004911019644749942"/>
+    <!-- PLACEHOLDER inertia, not CAD-exact (CAD ~1.2e-7..2.3e-7 was rounded to 0 by the
+         exporter). Physically valid; kept unchanged. See docs/URDF_INERTIA_AUDIT.md -->
     <inertia ixx="1e-6" iyy="1e-6" izz="1e-6" ixy="0.0" iyz="0.0" ixz="-0.0"/>
   </inertial>
@@ -394,4 +421,6 @@
     <origin xyz="-0.00029692851867108017 1.9537843565231583e-13 -9.71445146547012e-17" rpy="0 0 0"/>
     <mass value="0.004911019644749942"/>
+    <!-- PLACEHOLDER inertia, not CAD-exact (CAD ~1.2e-7..2.3e-7 was rounded to 0 by the
+         exporter). Physically valid; kept unchanged. See docs/URDF_INERTIA_AUDIT.md -->
     <inertia ixx="1e-6" iyy="1e-6" izz="1e-6" ixy="0.0" iyz="0.0" ixz="0.0"/>
   </inertial>
@@ -414,4 +443,6 @@
     <origin xyz="0.00029692851867092057 1.9551027463649007e-13 -1.3877787807814457e-16" rpy="0 0 0"/>
     <mass value="0.004911019644749942"/>
+    <!-- PLACEHOLDER inertia, not CAD-exact (CAD ~1.2e-7..2.3e-7 was rounded to 0 by the
+         exporter). Physically valid; kept unchanged. See docs/URDF_INERTIA_AUDIT.md -->
     <inertia ixx="1e-6" iyy="1e-6" izz="1e-6" ixy="-0.0" iyz="0.0" ixz="-0.0"/>
   </inertial>
@@ -434,4 +465,6 @@
     <origin xyz="0.0002969285186709657 1.952465966681416e-13 -8.326672684688674e-17" rpy="0 0 0"/>
     <mass value="0.004911019644749942"/>
+    <!-- PLACEHOLDER inertia, not CAD-exact (CAD ~1.2e-7..2.3e-7 was rounded to 0 by the
+         exporter). Physically valid; kept unchanged. See docs/URDF_INERTIA_AUDIT.md -->
     <inertia ixx="1e-6" iyy="1e-6" izz="1e-6" ixy="-0.0" iyz="0.0" ixz="-0.0"/>
   </inertial>
@@ -779,3 +812,41 @@
   <child link="top_1"/>
 </joint>
+<!-- ==========================================================================
+     lidar_link: added for simulation. It is NOT part of the Fusion 360 export and no
+     lidar CAD exists. The mount pose comes from the measured meshes (see
+     docs/SPIDERX_URDF_AUDIT.md): centred on the top plate (x=0.051, y=-0.045), body
+     resting on the plate's top surface (z=0.111), scan plane 0.030 m above it.
+     Yawed +90 deg so lidar_link +x points to the robot's front, which is +y of
+     base_link (base_link is not REP-103 aligned, audit item T1).
+     Replace the pose with the real mount/CAD when available.
+     ========================================================================== -->
+<link name="lidar_link">
+  <inertial>
+    <!-- SIMULATION_ESTIMATE: 0.17 kg (nominal RPLidar A1-class mass, not weighed) as a
+         solid cylinder r=0.035 m, h=0.040 m. See docs/URDF_INERTIA_AUDIT.md -->
+    <origin xyz="0 0 -0.010" rpy="0 0 0"/>
+    <mass value="0.17"/>
+    <inertia ixx="7.47e-05" iyy="7.47e-05" izz="1.041e-04" ixy="0.0" iyz="0.0" ixz="0.0"/>
+  </inertial>
+  <visual>
+    <origin xyz="0 0 -0.010" rpy="0 0 0"/>
+    <geometry>
+      <cylinder radius="0.035" length="0.040"/>
+    </geometry>
+    <material name="lidar_black">
+      <color rgba="0.100 0.100 0.100 1.000"/>
+    </material>
+  </visual>
+  <collision>
+    <origin xyz="0 0 -0.010" rpy="0 0 0"/>
+    <geometry>
+      <cylinder radius="0.035" length="0.040"/>
+    </geometry>
+  </collision>
+</link>
+<joint name="lidar_joint" type="fixed">
+  <origin xyz="0.051 -0.045 0.141" rpy="0 0 1.5707963267948966"/>
+  <parent link="base_link"/>
+  <child link="lidar_link"/>
+</joint>
 </robot>

Commit message: spiderx_description: optional Fortress ros2_control block (enable_control:=false default)
Adds spiderx_fortress_control.xacro (gz_ros2_control/GazeboSimSystem, 12 joints,
command=position, state=position+velocity) and a control-mode bridge that omits
joint_states so there is exactly one /joint_states publisher. The passive
description is byte-identical when enable_control is false.

Co-Authored-By: Claude Opus 5.5 <noreply@anthropic.com>
Claude-Session: https://claude.ai/code/session_01QzFL2kguRig19KtzFfqEm3

File: src/spiderx_description/urdf/spiderx.urdf.xacro (robot description, xacro)
@@ -13,4 +13,16 @@
   ${xacro.fatal("sim_backend must be 'classic', 'fortress' or 'none', got '" + sim_backend + "'")}
 </xacro:unless>
+<!-- enable_control (M1): add gz_ros2_control joint position control (fortress only).
+     controllers_file: absolute path of the ros2_control controller YAML (set by the launch file).
+     Default false keeps the verified passive simulation unchanged. -->
+<xacro:arg name="enable_control" default="false" />
+<xacro:arg name="controllers_file" default="" />
+<xacro:property name="enable_control" value="$(arg enable_control)" />
+<xacro:if value="${enable_control and sim_backend != 'fortress'}">
+  ${xacro.fatal("enable_control:=true is only supported with sim_backend:=fortress")}
+</xacro:if>
+<xacro:if value="${enable_control and '$(arg controllers_file)' == ''}">
+  ${xacro.fatal("enable_control:=true requires controllers_file:=/absolute/path/to/controllers.yaml")}
+</xacro:if>
 <xacro:include filename="$(find spiderx_description)/urdf/materials.xacro" />
 <xacro:if value="${sim_backend == 'classic'}">
@@ -20,4 +32,7 @@
 <xacro:if value="${sim_backend == 'fortress'}">
   <xacro:include filename="$(find spiderx_description)/urdf/spiderx_fortress.gazebo.xacro" />
+</xacro:if>
+<xacro:if value="${sim_backend == 'fortress' and enable_control}">
+  <xacro:include filename="$(find spiderx_description)/urdf/spiderx_fortress_control.xacro" />
 </xacro:if>
 <link name="dummy_link">

File: src/spiderx_description/urdf/spiderx_fortress.gazebo.xacro (robot description, xacro)
@@ -54,13 +54,17 @@
     </sensor>
   </gazebo>
+  <!-- enable_control:=true (M1) omits this system, because joint_state_broadcaster
+       (gz_ros2_control) publishes /joint_states instead. Exactly one publisher either way. -->
+  <xacro:unless value="$(arg enable_control)">
   <!-- Publishes the state of every model joint as measured by the physics engine.
        The launch file bridges this to /joint_states, which robot_state_publisher uses
        for the leg TF. Nothing here commands the joints: the model is passive. -->
-  <gazebo>
-    <plugin filename="ignition-gazebo-joint-state-publisher-system"
-            name="ignition::gazebo::systems::JointStatePublisher">
-      <topic>${gz_joint_state_topic}</topic>
-    </plugin>
-  </gazebo>
+    <gazebo>
+      <plugin filename="ignition-gazebo-joint-state-publisher-system"
+              name="ignition::gazebo::systems::JointStatePublisher">
+        <topic>${gz_joint_state_topic}</topic>
+      </plugin>
+    </gazebo>
+  </xacro:unless>
   <!-- Contact parameters kept identical to the legacy Classic file (spiderx.gazebo):
        mu1 = mu2 = 0.2 and self_collide = false on the same 30 CAD links. These are the
